Commit message: ADD: add partial config

File: resources/robots/g1/urdf/g1_full.urdf (robot description, URDF)
Before this commit: robot g1, 44 links, 43 joints
Joints:
- joint left_elbow_pitch_joint: type fixed -> revolute
- joint left_elbow_roll_joint: type fixed -> revolute
- joint left_five_joint: type fixed -> revolute
- joint left_four_joint: type fixed -> revolute
- joint left_one_joint: type fixed -> revolute
- joint left_shoulder_pitch_joint: type fixed -> revolute
- joint left_shoulder_roll_joint: type fixed -> revolute
- joint left_shoulder_yaw_joint: type fixed -> revolute
- joint left_six_joint: type fixed -> revolute
- joint left_three_joint: type fixed -> revolute
- joint left_two_joint: type fixed -> revolute
- joint left_zero_joint: type fixed -> revolute
- joint right_elbow_pitch_joint: type fixed -> revolute
- joint right_elbow_roll_joint: type fixed -> revolute
- joint right_five_joint: type fixed -> revolute
- joint right_four_joint: type fixed -> revolute
- joint right_one_joint: type fixed -> revolute
- joint right_shoulder_pitch_joint: type fixed -> revolute
- joint right_shoulder_roll_joint: type fixed -> revolute
- joint right_shoulder_yaw_joint: type fixed -> revolute
- joint right_six_joint: type fixed -> revolute
- joint right_three_joint: type fixed -> revolute
- joint right_two_joint: type fixed -> revolute
- joint right_zero_joint: type fixed -> revolute
- joint torso_joint: type fixed -> revolute
