Commit message: ADD: separate different robot config

File: resources/robots/g1/urdf/g1_leg.urdf (robot description, URDF)
Before this commit: robot g1, 44 links, 43 joints
Joints:
- joint left_elbow_pitch_joint: type revolute -> fixed
- joint left_elbow_roll_joint: type revolute -> fixed
- joint left_five_joint: type revolute -> fixed
- joint left_four_joint: type revolute -> fixed
- joint left_one_joint: type revolute -> fixed
- joint left_shoulder_pitch_joint: type revolute -> fixed
- joint left_shoulder_roll_joint: type revolute -> fixed
- joint left_shoulder_yaw_joint: type revolute -> fixed
- joint left_six_joint: type revolute -> fixed
- joint left_three_joint: type revolute -> fixed
- joint left_two_joint: type revolute -> fixed
- joint left_zero_joint: type revolute -> fixed
- joint right_elbow_pitch_joint: type revolute -> fixed
- joint right_elbow_roll_joint: type revolute -> fixed
- joint right_five_joint: type revolute -> fixed
- joint right_four_joint: type revolute -> fixed
- joint right_one_joint: type revolute -> fixed
- joint right_shoulder_pitch_joint: type revolute -> fixed
- joint right_shoulder_roll_joint: type revolute -> fixed
- joint right_shoulder_yaw_joint: type revolute -> fixed
- joint right_six_joint: type revolute -> fixed
- joint right_three_joint: type revolute -> fixed
- joint right_two_joint: type revolute -> fixed
- joint right_zero_joint: type revolute -> fixed
- joint torso_joint: type revolute -> fixed

File: resources/robots/g1/urdf/g1_leg_arm.urdf (robot description, URDF)
Before this commit: robot g1, 44 links, 43 joints
Joints:
- joint left_five_joint: type revolute -> fixed
- joint left_four_joint: type revolute -> fixed
- joint left_one_joint: type revolute -> fixed
- joint left_six_joint: type revolute -> fixed
- joint left_three_joint: type revolute -> fixed
- joint left_two_joint: type revolute -> fixed
- joint left_zero_joint: type revolute -> fixed
- joint right_five_joint: type revolute -> fixed
- joint right_four_joint: type revolute -> fixed
- joint right_one_joint: type revolute -> fixed
- joint right_six_joint: type revolute -> fixed
- joint right_three_joint: type revolute -> fixed
- joint right_two_joint: type revolute -> fixed
- joint right_zero_joint: type revolute -> fixed
- joint torso_joint: type revolute -> fixed
